Commit message: gazebo

File: description/example_gazebo.xacro (robot description, xacro)
@@ -35,5 +35,5 @@
         <plugin name="gazebo_ros_joint_pose_trajectory"
             filename="libgazebo_ros_joint_pose_trajectory.so">
-            <update_rate>2</update_rate>
+            <update_rate>20</update_rate>
         </plugin>
     </gazebo>
@@ -55,5 +55,5 @@
             try swapping "depth" to "camera"-->
     <gazebo reference="camera_link">
-        <sensor type="depth" name="my_camera">
+        <sensor type="camera" name="my_camera">  <!-- type="depth"-->
             <update_rate>20</update_rate>
             <visualize>true</visualize>

File: description/example_robot.urdf.xacro (robot description, xacro)
@@ -83,4 +83,5 @@
         <axis xyz="0 -1 0"/>
         <limit lower="0" upper="${pi/2}" velocity="100" effort="100"/>
+        <dynamics damping="10.0" friction="10.0"/>
     </joint>
     <!-- arm_link describes the arm -->
