Commit message: visual

File: description/bruinbot_core.xacro (robot description, xacro)
@@ -31,4 +31,10 @@
         <color rgba="1 0 0 1"/>
     </material>
+    <material name="ucla blue">
+        <color rgba="0.153 0.455 0.682 1"/>
+    </material>
+    <material name="ucla gold">
+        <color rgba="1 0.820 0 1"/>
+    </material>
     <!-- BASE LINK -->
     <link name="base_link">
@@ -54,5 +60,5 @@
                 <box size="${chassis_length} ${chassis_width} ${chassis_height}"/>
             </geometry>
-            <material name="orange"/>
+            <material name="ucla gold"/>
         </visual>
         <collision>
@@ -67,5 +73,5 @@
     </link>
     <gazebo reference="chassis">
-        <material>Gazebo/Orange</material>
+        <material>Gazebo/Yellow</material>
     </gazebo>
     <!-- LEFT WHEEL LINK -->
@@ -81,5 +87,5 @@
                 <cylinder radius="${wheel_radius}" length="${wheel_thickness}"/>
             </geometry>
-            <material name="blue"/>
+            <material name="ucla blue"/>
         </visual>
         <collision>
@@ -93,5 +99,5 @@
     </link>
     <gazebo reference="left_wheel">
-        <material>Gazebo/Blue</material>
+        <material>Gazebo/Turquoise</material>
     </gazebo>
     <!-- RIGHT WHEEL LINK -->
@@ -107,5 +113,5 @@
                 <cylinder radius="${wheel_radius}" length="${wheel_thickness}"/>
             </geometry>
-            <material name="blue"/>
+            <material name="ucla blue"/>
         </visual>
         <collision>
@@ -119,5 +125,5 @@
     </link>
     <gazebo reference="right_wheel">
-        <material>Gazebo/Blue</material>
+        <material>Gazebo/Turquoise</material>
     </gazebo>
     <!-- CASTER WHEEL LINK -->

File: description/bruinbot_lidar.xacro (robot description, xacro)
@@ -11,5 +11,5 @@
                 <cylinder radius="0.05" length="0.04"/>
             </geometry>
-            <material name="red"/>
+            <material name="ucla blue"/>
         </visual>
         <collision>
@@ -23,5 +23,5 @@
     </link>
     <gazebo reference="laser_frame">
-        <material>Gazebo/Red</material>
+        <material>Gazebo/Turquoise</material>
         <sensor name="laser" type="ray">
             <pose> 0 0 0 0 0 0 </pose>
